File: Hardware/Yavia_Carrier/Yavia_Carrier.kicad_sch (KiCad schematic)
At the start: 42 parts, among them J1 Power, J2 Serial, J3 52610-1572, J4 STRB_IS, J5 STRB, J6 52610-1572, J7 FLASH, Q1 MMBT2222ALT1G, U1 RaspberryPi-CM-_SOM, U2 AP63203, U3 LM3671, U4 TCMT1103, U5 LDD600L, U6 74AHC1G32, U8 Yavia_GND, U9 Yavia

Commit message: add one MIPI CSI connection
Parts:
- added C36, C37, C38, C39, C40: 22uF, Capacitor_SMD:C_0603_1608Metric_Pad1.05x0.95mm_HandSolder, symbol RPI-Carrier-rescue:C_Small-Device
- added J10: 52610-1572, RPi-Carrier:526101572, symbol RPICarrier:52610-1572
- added L5, L6: 330 ohm/1.7A, symbol Device:L
- added R27: 10m, Resistor_SMD:R_0603_1608Metric_Pad1.05x0.95mm_HandSolder, symbol RPI-Carrier-rescue:R_Small-Device
- added U10, U12: Verdin iMX8M Plus, Yavia_carrier:2309409-2, symbol RPICarrier:RaspberryPi-CM-_SOM
- added U11: Verdin iMX8M Plus, Yavia_Carrier: 2309409-2, symbol RPICarrier:RaspberryPi-CM-_SOM
- U8: value Yavia_GND -> Verdin iMX8M Plus; footprint RPi-Carrier:1473005-4 -> Yavia_carrier:2309409-2; manf# 1473005-4 -> 2309409-2
- U9: value Yavia -> Verdin iMX8M Plus; footprint RPi-Carrier:1473005-4 -> Yavia_carrier:2309409-2; manf# 1473005-4 -> 2309409-2
Connections:
- net +3V3: now also J10.1
- net +5V: now also L5.1, L6.1
- net CAM0_CLK+: now also J10.13
- net CAM0_CLK-: now also J10.15
- net CAM0_D0+: now also J10.25
- net CAM0_D0-: now also J10.27
- net CAM0_D1+: now also J10.19
- net CAM0_D1-: now also J10.21
- net CAM0_IO0: now also J10.9, U10.206 (GPIO_1)
- net CAM0_IO1: now also J10.7, U10.208 (GPIO_2)
- net CAM0_SCL: now also U9.14 (I2C_1_SCL), J10.5
- net CAM0_SDA: now also U9.12 (I2C_1_SDA), J10.3
- net CAM1_CLK+: now also U12.111 (CSI_1_CLK_P)
- net CAM1_CLK-: now also U12.113 (CSI_1_CLK_N)
- net CAM1_D0+: now also U12.123 (CSI_1_D0_P)
- net CAM1_D0-: now also U12.125 (CSI_1_D0_N)
- net CAM1_D1+: now also U12.117 (CSI_1_D1_P)
- net CAM1_D1-: now also U12.119 (CSI_1_D1_N)
- net CAM1_D2+: now also U12.105 (CSI_1_D2_P)
- net CAM1_D2-: now also U12.107 (CSI_1_D2_N)
- net CAM1_D3+: now also U12.99 (CSI_1_D3_P)
- net CAM1_D3-: now also U12.101 (CSI_1_D3_N)
- net CAM1_IO0: now also U10.212 (GPIO_4)
- net CAM1_IO1: now also U10.210 (GPIO_3)
- net CAM1_SCL: now also U9.93 (I2C_4_CSI_SDA)
- net CAM1_SDA: now also U9.95 (I2C_4_CSI_SCL)
- net Flash_EN: now also U10.222 (GPIO_8)
- net GND: now also C36.2, C37.2, C38.2, C39.2, C40.2, J10.11, J10.17, J10.23, J10.29
- net LED_R: now also U10.220 (GPIO_7)
- net RX_UART: now also U9.129 (UART_1_RXD)
- net TX_UART: now also U9.131 (UART_1_TXD)
- new net: L5.2, L6.2, R27.1
- new net VT: C36.1, C37.1, C38.1, C39.1, C40.1, R27.2, U11.251 (VCC), U11.253 (VCC), U11.255 (VCC), U11.257 (VCC), U11.259 (VCC)
Other:
- moved on the sheet: U1I

Commit message: add MIPI SCI and power supply connections,
Parts:
- removed J10: 52610-1572, RPi-Carrier:526101572, symbol RPICarrier:52610-1572
- removed R2: 1K, Resistor_SMD:R_0603_1608Metric_Pad1.05x0.95mm_HandSolder, symbol RPI-Carrier-rescue:R_Small-Device
- removed unit 6 of U1
- removed unit 2 of U1
- removed unit 3 of U1
- removed unit 4 of U1
- removed unit 1 of U1
- removed unit 8 of U1
- U1: value RaspberryPi-CM-_SOM -> Verdin iMX8M Plus; footprint RPi-Carrier:1473005-4 -> Yavia_carrier:2309409-2; manf# 1473005-4 -> 2309409-2
- U1: renamed from U11; footprint Yavia_Carrier: 2309409-2 -> Yavia_carrier:2309409-2
- renumbered U12 to U1, U9 to U1, U8 to U1, U10 to U1
Connections:
- net CAM0_CLK+: now also U1.162 (CSI2_CLK_P)
- net CAM0_CLK-: now also U1.160 (CSI2_CLK_N)
- net CAM0_D0+: now also U1.150 (CSI2_D0_P)
- net CAM0_D0-: now also U1.148 (CSI2_D0_N)
- net CAM0_D1+: now also U1.156 (CSI2_D1_P)
- net CAM0_D1-: now also U1.154 (CSI2_D1_N)
- net CAM0_IO0: now also U1.216 (GPIO_5); no longer U1.206 (GPIO_1)
- net CAM0_IO1: now also U1.218 (GPIO_6); no longer U1.208 (GPIO_2)
- net CAM1_CLK+: no longer U1.147 (CAM1_CP)
- net CAM1_CLK-: no longer U1.149 (CAM1_CN)
- net CAM1_D0+: no longer U1.159 (CAM1_DP0)
- net CAM1_D0-: no longer U1.161 (CAM1_DN0)
- net CAM1_D1+: no longer U1.153 (CAM1_DP1)
- net CAM1_D1-: no longer U1.155 (CAM1_DN1)
- net CAM1_D2+: no longer U1.141 (CAM1_DP2)
- net CAM1_D2-: no longer U1.143 (CAM1_DN2)
- net CAM1_D3+: no longer U1.135 (CAM1_DP3)
- net CAM1_D3-: no longer U1.137 (CAM1_DN3)
- net CAM1_IO0: now also U1.222 (GPIO_8); no longer U1.212 (GPIO_4)
- net CAM1_IO1: now also U1.220 (GPIO_7); no longer U1.210 (GPIO_3)
- net Flash_EN: now also U1.208 (GPIO_2); no longer U1.222 (GPIO_8)
- net GND: no longer U1.71 (GND)
- net LED_R: now also U1.206 (GPIO_1); no longer U1.220 (GPIO_7)
- no-connect marks 37 -> 191
Other:
- note removed: "Check startup sequence"
- moved on the sheet: C11, C12, C13, C36, C37, C38, C39, C4, C40, C5, C7, D2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

Commit message: add ldd circuit
Parts:
- added J10: STRB_IS, Connector_PinHeader_2.54mm:PinHeader_1x02_P2.54mm_Vertical, symbol RPI-Carrier-rescue:Screw_Terminal_01x02-Connector
- added J11: STRB, Connector_PinHeader_2.54mm:PinHeader_1x02_P2.54mm_Vertical, symbol RPI-Carrier-rescue:Screw_Terminal_01x02-Connector
- added J12: FLASH, Connector_PinHeader_2.54mm:PinHeader_1x02_P2.54mm_Vertical, symbol RPI-Carrier-rescue:Conn_01x02_Female-Connector
- added Q2: MMBT2222ALT1G, Package_TO_SOT_SMD:SOT-23, symbol RPI-Carrier-rescue:MMBT3904-Transistor_BJT
- added R27, R29: 1K, Resistor_SMD:R_0603_1608Metric_Pad1.05x0.95mm_HandSolder, symbol RPI-Carrier-rescue:R_Small-Device
- added R28: 500K, Resistor_SMD:R_0603_1608Metric_Pad1.05x0.95mm_HandSolder, symbol RPI-Carrier-rescue:R_Small-Device
- added R30: 10K, Resistor_SMD:R_0603_1608Metric_Pad1.05x0.95mm_HandSolder, symbol RPI-Carrier-rescue:R_Small-Device
- added U10: LDD600L, RPi-Carrier:LDD-L, symbol RPICarrier:LDD500L
- added U11: 74AHC1G32, Package_TO_SOT_SMD:SOT-23-5, symbol RPI-Carrier-rescue:74AHC1G32-74xGxx
- added U9: TCMT1103, Package_SO:SOP-4_4.4x2.6mm_P1.27mm, symbol RPI-Carrier-rescue:TCMT1103-Isolator
- renumbered C36 to C1, C8 to C10, C9 to C11, C10 to C12, C7 to C13, C11 to C14, C5 to C15, C4 to C16, C12 to C17, C13 to C18, C1 to C2, C37 to C3, C38 to C4, C39 to C5, C2 to C6, C3 to C7, C40 to C8, C6 to C9, J4 to J3, J5 to J4, J3 to J5, L5 to L1, L6 to L2, L1 to L3, L2 to L4, R27 to R2, U4 to U5, U5 to U6, U6 to U7
Connections:
- net +12V: now also R30.1, U10.1 (VIN+)
- net +36V: now also J12.1 (Pin_1), U10.6 (+VOUT)
- net +3V3: now also R28.1, U11.5 (VCC)
- net GND: now also J10.1 (Pin_1), Q2.2 (E), U10.4 (VIN-), U11.3 (GND), U9.3
- net GNDPWR: now also J12.2 (Pin_2), U10.5 (-VOUT)
- net LDD_OUT: now also Q1.3 (C), R9.2
- net Flash_EN_1: now reaches U1.210 (GPIO_3)
- net Flash_EN_1: now also U11.2
- new net: Q2.1 (B), R29.1
- new net: R29.2, U11.4
- new net: R27.1, U9.2
- new net: J11.1 (Pin_1), R27.2
- new net: J11.2 (Pin_2), U9.1
- new net LDD_OUT_1: Q2.3 (C), R30.2, U10.3 (PWM)
- new net opto_out_1: J10.2 (Pin_2), R28.2, U11.1, U9.4
- no-connect marks 191 -> 190
Other:
- note added: "Camera Flash input 1"
- note added: "Camera Flash input 2"
- note removed: "Camera Flash input"
- moved on the sheet: J7, Q1, R8, R9, U6, U7

Commit message: Fix U1 symbol & started pcb
Parts:
- removed U1 (x2): Verdin iMX8M Plus, Yavia_carrier:2309409-2, symbol RPICarrier:RaspberryPi-CM-_SOM
- added U1: Verdin iMX8M Plus, Yavia_carrier:23094092, symbol Verdin iMX8M Plus:Yavia_carrier
- C1, C10, C11, C12, C13, C14, C15, C16, C17, C18, C3, C4, C5, C6, C7, C8, C9: footprint Capacitor_SMD:C_0603_1608Metric_Pad1.05x0.95mm_HandSolder -> Capacitor_SMD:C_0603_1608Metric_Pad1.08x0.95mm_HandSolder
- J1: footprint RPi-Carrier:DF11CZ-6DP-2V -> Yavia_carrier:DF11CZ-6DP-2V
- J10: renamed from J6; footprint RPi-Carrier:526101572 -> Yavia_carrier:526101572
- J7: renamed from J5; footprint RPi-Carrier:526101572 -> Yavia_carrier:526101572
- R1, R2, R3, R4, R5, R6: footprint Resistor_SMD:R_0603_1608Metric_Pad1.05x0.95mm_HandSolder -> Resistor_SMD:R_0603_1608Metric_Pad0.98x0.95mm_HandSolder
- R10: renamed from R8; footprint Resistor_SMD:R_0603_1608Metric_Pad1.05x0.95mm_HandSolder -> Resistor_SMD:R_0603_1608Metric_Pad0.98x0.95mm_HandSolder
- R11: renamed from R29; footprint Resistor_SMD:R_0603_1608Metric_Pad1.05x0.95mm_HandSolder -> Resistor_SMD:R_0603_1608Metric_Pad0.98x0.95mm_HandSolder
- R12: renamed from R9; footprint Resistor_SMD:R_0603_1608Metric_Pad1.05x0.95mm_HandSolder -> Resistor_SMD:R_0603_1608Metric_Pad0.98x0.95mm_HandSolder
- R13: renamed from R30; footprint Resistor_SMD:R_0603_1608Metric_Pad1.05x0.95mm_HandSolder -> Resistor_SMD:R_0603_1608Metric_Pad0.98x0.95mm_HandSolder
- R7: renamed from R27; footprint Resistor_SMD:R_0603_1608Metric_Pad1.05x0.95mm_HandSolder -> Resistor_SMD:R_0603_1608Metric_Pad0.98x0.95mm_HandSolder
- R8: renamed from R7; footprint Resistor_SMD:R_0603_1608Metric_Pad1.05x0.95mm_HandSolder -> Resistor_SMD:R_0603_1608Metric_Pad0.98x0.95mm_HandSolder
- R9: renamed from R28; footprint Resistor_SMD:R_0603_1608Metric_Pad1.05x0.95mm_HandSolder -> Resistor_SMD:R_0603_1608Metric_Pad0.98x0.95mm_HandSolder
- U6: footprint RPi-Carrier:LDD-L -> Yavia_carrier:LDD-L
- U7: renamed from U10; footprint RPi-Carrier:LDD-L -> Yavia_carrier:LDD-L
- renumbered J10 to J4, J4 to J5, J11 to J6, J7 to J8, J12 to J9, U5 to U4, U9 to U5, U7 to U8, U11 to U9
Connections:
- net +3V3: now also J10.2
- net CAM0_CLK+: now also J10.14, U1.162 (CSI2_CLK_P)
- net CAM0_CLK-: now also J10.16, U1.160 (CSI2_CLK_N)
- net CAM0_D0+: now also J10.26, U1.150 (CSI2_D0_P)
- net CAM0_D0-: now also J10.28, U1.148 (CSI2_D0_N)
- net CAM0_D1+: now also J10.20, U1.156 (CSI2_D1_P)
- net CAM0_D1-: now also J10.22, U1.154 (CSI2_D1_N)
- net CAM0_IO0: now also J10.10, U1.216 (GPIO_5)
- net CAM0_IO1: now also J10.8, U1.218 (GPIO_6)
- net CAM0_SCL: now also J10.6, U1.14 (I2C_1_SCL)
- net CAM0_SDA: now also J10.4, U1.12 (I2C_1_SDA)
- net CAM1_CLK+: now also U1.111 (CSI_1_CLK_P)
- net CAM1_CLK-: now also U1.113 (CSI_1_CLK_N)
- net CAM1_D0+: now also U1.123 (CSI_1_D0_P)
- net CAM1_D0-: now also U1.125 (CSI_1_D0_N)
- net CAM1_D1+: now also U1.117 (CSI_1_D1_P)
- net CAM1_D1-: now also U1.119 (CSI_1_D1_N)
- net CAM1_D2+: now also U1.105 (CSI_1_D2_P)
- net CAM1_D2-: now also U1.107 (CSI_1_D2_N)
- net CAM1_D3+: now also U1.99 (CSI_1_D3_P)
- net CAM1_D3-: now also U1.101 (CSI_1_D3_N)
- net CAM1_IO0: now also U1.222 (GPIO_8)
- net CAM1_IO1: now also U1.220 (GPIO_7)
- net CAM1_SCL: now also U1.93 (I2C_4_CSI_SDA)
- net CAM1_SDA: now also U1.95 (I2C_4_CSI_SCL)
- net Flash_EN: now also U1.208 (GPIO_2)
- net Flash_EN_1: now also U1.210 (GPIO_3)
- net GND: now also J10.12, J10.18, J10.24, J10.30, U1.10 (GND), U1.103 (GND), U1.109 (GND), U1.11 (GND), U1.110 (GND), U1.115 (GND), U1.121 (GND), U1.122 (GND), U1.127 (GND), U1.134 (GND), U1.145 (GND), U1.146 (GND), U1.158 (GND), U1.167 (GND), U1.170 (GND), U1.173 (GND), U1.179 (GND), U1.18 (GND), U1.182 (GND), U1.194 (GND), U1.195 (GND), U1.204 (GND), U1.209 (GND), U1.223 (GND), U1.224 (GND), U1.229 (GND), U1.230 (GND), U1.236 (GND), U1.242 (GND), U1.243 (GND), U1.27 (GND), U1.28 (GND), U1.33 (GND), U1.39 (GND), U1.40 (GND), U1.45 (GND), U1.50 (GND), U1.51 (GND), U1.65 (GND), U1.68 (GND), U1.71 (GND), U1.77 (GND), U1.83 (GND), U1.86 (GND), U1.89 (GND), U1.97 (GND), U1.98 (GND)
- net LED_R: now also U1.206 (GPIO_1)
- net RX_UART: now also U1.129 (UART_1_RXD)
- net TX_UART: now also U1.131 (UART_1_TXD)
- net UP-D+: now also U1.165 (USB_1_ID)
- net UP-D-: now also U1.163 (USB_1_D_N)
- net VT: now also U1.251 (VCC), U1.253 (VCC), U1.255 (VCC), U1.257 (VCC), U1.259 (VCC)
- no-connect marks 190 -> 189
Other:
- moved on the sheet: C17, C18, J10, J7
